Commit message: Add files via upload

File: mis_modelos_robots/urdf/turtlebot_completo.urdf (robot description, URDF)
Before this commit: robot turtlebot_visual, 30 links, 29 joints
Links:
- link base_link: geometry collision cylinder length=0.10938 radius=0.178; visual mesh filename=package://mis_modelos_robots/meshes/kobuki_meshes/main_body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
- link camera_link: geometry collision box size=0.0730 0.2760 0.0720; visual mesh filename=package://mis_modelos_robots/meshes/kinect.dae
- link laser_sensor_link: geometry visual mesh filename=package://mis_modelos_robots/meshes/kobuki_meshes/sensors/h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
- link plate_bottom_link: geometry collision cylinder length=0.006 radius=0.170; visual mesh filename=package://mis_modelos_robots/meshes/kobuki_meshes/stacks/he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
- link plate_middle_link: geometry collision cylinder length=0.006 radius=0.170; visual mesh filename=package://mis_modelos_robots/meshes/kobuki_meshes/stacks/he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
- link plate_top_link: geometry collision cylinder length=0.006 radius=0.170; visual mesh filename=package://mis_modelos_robots/meshes/kobuki_meshes/stacks/he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
- link pole_bottom_0_link: geometry collision cylinder length=0.0492 radius=0.006; visual mesh filename=package://mis_modelos_robots/meshes/kobuki_meshes/stacks/he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
- link pole_bottom_1_link: geometry collision cylinder length=0.0492 radius=0.006; visual mesh filename=package://mis_modelos_robots/meshes/kobuki_meshes/stacks/he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
- link pole_bottom_2_link: geometry collision cylinder length=0.0492 radius=0.006; visual mesh filename=package://mis_modelos_robots/meshes/kobuki_meshes/stacks/he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
- link pole_bottom_3_link: geometry collision cylinder length=0.0492 radius=0.006; visual mesh filename=package://mis_modelos_robots/meshes/kobuki_meshes/stacks/he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
- link pole_bottom_4_link: geometry collision cylinder length=0.0492 radius=0.006; visual mesh filename=package://mis_modelos_robots/meshes/kobuki_meshes/stacks/he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
- link pole_bottom_5_link: geometry collision cylinder length=0.0492 radius=0.006; visual mesh filename=package://mis_modelos_robots/meshes/kobuki_meshes/stacks/he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
- link pole_middle_0_link: geometry collision cylinder length=0.0608 radius=0.006; visual mesh filename=package://mis_modelos_robots/meshes/kobuki_meshes/stacks/he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
- link pole_middle_1_link: geometry collision cylinder length=0.0608 radius=0.006; visual mesh filename=package://mis_modelos_robots/meshes/kobuki_meshes/stacks/he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
- link pole_middle_2_link: geometry collision cylinder length=0.0608 radius=0.006; visual mesh filename=package://mis_modelos_robots/meshes/kobuki_meshes/stacks/he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
- link pole_middle_3_link: geometry collision cylinder length=0.0608 radius=0.006; visual mesh filename=package://mis_modelos_robots/meshes/kobuki_meshes/stacks/he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
- link pole_top_0_link: geometry collision cylinder length=0.2032 radius=0.006; visual mesh filename=package://mis_modelos_robots/meshes/kobuki_meshes/stacks/he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
- link pole_top_1_link: geometry collision cylinder length=0.2032 radius=0.006; visual mesh filename=package://mis_modelos_robots/meshes/kobuki_meshes/stacks/he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
- link pole_top_2_link: geometry collision cylinder length=0.2032 radius=0.006; visual mesh filename=package://mis_modelos_robots/meshes/kobuki_meshes/stacks/he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
- link pole_top_3_link: geometry collision cylinder length=0.2032 radius=0.006; visual mesh filename=package://mis_modelos_robots/meshes/kobuki_meshes/stacks/he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
- link wheel_left_link: geometry collision cylinder length=0.0206 radius=0.0350; visual mesh filename=package://mis_modelos_robots/meshes/kobuki_meshes/wheel.dae
- link wheel_right_link: geometry collision cylinder length=0.0206 radius=0.0350; visual mesh filename=package://mis_modelos_robots/meshes/kobuki_meshes/wheel.dae
