Commit message: Add files via upload

File: mis_modelos_robots/urdf/trabajo_urdf.urdf (robot description, URDF)
Before this commit: robot mi_primer_robot, 3 links, 2 joints
Links:
- removed link wheel_left_link
- removed link wheel_right_link
- added link left_wheel, mass 5; collision box size=0.5 0.5 0.25; visual cylinder length=0.1 radius=0.2
- added link right_wheel, mass 5; collision box size=0.5 0.5 0.25; visual cylinder length=0.1 radius=0.2
- link base_link: mass None -> 5; geometry collision box size=0.5 0.5 0.25; visual box size=0.5 0.5 0.25
Joints:
- removed joint wheel_left_joint
- removed joint wheel_right_joint
- added joint joint_left_wheel: type continuous, parent base_link, child left_wheel, origin xyz=0 0.30 0 rpy=0 0 0, axis 0 1 0
- added joint joint_right_wheel: type continuous, parent base_link, child right_wheel, origin xyz=0 -0.30 0 rpy=0 0 0, axis 0 1 0
