Commit message: Add files via upload

File: mis_modelos_robots/urdf/mi_primer_robot.urdf (robot description, URDF)
Before this commit: robot mi_primer_robot, 5 links, 5 joints
Links:
- removed link base_link
- removed link camera_link
- removed link head_link
- removed link left_eye_link
- removed link right_eye_link
- added link link_chassis, mass 5; collision box size=0.5 0.3 0.07; collision sphere radius=0.05
- added link link_left_wheel, mass 0.2; collision cylinder length=0.04 radius=0.1; visual cylinder length=0.04 radius=0.1
- added link link_right_wheel, mass 0.2; collision cylinder length=0.04 radius=0.1; visual cylinder length=0.04 radius=0.1
- added link sensor_laser, mass 1; collision cylinder length=0.1 radius=0.05; visual cylinder length=0.1 radius=0.05
Joints:
- removed joint base_head_joint
- removed joint camera_joint
- removed joint head_roll_joint
- removed joint left_eye_joint
- removed joint right_eye_joint
- added joint joint_left_wheel: type continuous, parent link_chassis, child link_left_wheel, origin xyz=-0.05 -0.15 0 rpy=0 0 0, axis 0 1 0, limit effort=10000 velocity=1000
- added joint joint_right_wheel: type continuous, parent link_chassis, child link_right_wheel, origin xyz=-0.05 0.15 0 rpy=0 0 0, axis 0 1 0, limit effort=10000 velocity=1000
- added joint joint_sensor_laser: type fixed, parent link_chassis, child sensor_laser, origin xyz=0.15 0 0.05 rpy=0 0 0

File: mis_modelos_robots/urdf/trabajo_urdf.urdf (robot description, URDF)
Before this commit: robot trabajo_urdf, 3 links, 2 joints
Links:
- removed link base_link
- removed link left_wheel
- removed link right_wheel
- added link link_chassis, mass 5; collision box size=0.5 0.3 0.07; collision sphere radius=0.05
- added link link_left_wheel, mass 0.2; collision cylinder length=0.04 radius=0.1; visual cylinder length=0.04 radius=0.1
- added link link_right_wheel, mass 0.2; collision cylinder length=0.04 radius=0.1; visual cylinder length=0.04 radius=0.1
- added link sensor_laser, mass 1; collision cylinder length=0.1 radius=0.05; visual cylinder length=0.1 radius=0.05
Joints:
- added joint joint_sensor_laser: type fixed, parent link_chassis, child sensor_laser, origin xyz=0.15 0 0.05 rpy=0 0 0
- joint joint_left_wheel: child left_wheel -> link_left_wheel; limit (none) -> effort=10000 velocity=1000; origin xyz=0 0.30 0 rpy=0 0 0 -> xyz=-0.05 -0.15 0 rpy=0 0 0; parent base_link -> link_chassis
- joint joint_right_wheel: child right_wheel -> link_right_wheel; limit (none) -> effort=10000 velocity=1000; origin xyz=0 -0.30 0 rpy=0 0 0 -> xyz=-0.05 0.15 0 rpy=0 0 0; parent base_link -> link_chassis
